File: Rev A.brd (EAGLE design)
At the start: 160 x 100 mm, 38 parts, among them IC2 NE555, IC3 LM358N, Q2 TIP41C

Commit message: Finished the layout
Parts:
- removed C1: 47uF, rcl:E2,5-6
- removed ON: (no value), led:LED2X5
- removed R8: 1kΩ, resistor:0207/10
- added R14, R15: 100kΩ, resistor:0207/10
- moved CURR_SENSE 159.7 mm to (54.6, 5.08), turned to 180 degrees
- moved R5 136.9 mm to (64.8, 19.1), turned to 90 degrees
- moved R2 131.3 mm to (49.5, 19.1), turned to 90 degrees
- moved R10 125.5 mm to (20.3, 21.6), turned to 270 degrees
- moved C2 121.8 mm to (35.6, 21.6), turned to 270 degrees
- moved R4 117.0 mm to (59.7, 19.1), turned to 90 degrees
- moved R9 113.5 mm to (17.8, 21.6), turned to 270 degrees
- moved RNG_SEL 111.9 mm to (19.1, 12.7), turned to 180 degrees
- moved R1 110.9 mm to (44.5, 19.1), turned to 90 degrees
- moved C3 109.3 mm to (6.35, 14.0)
- moved R3 98.4 mm to (54.6, 19.1), turned to 90 degrees
- moved Q2 93.7 mm to (41.9, 41.9)
- moved R11 90.3 mm to (22.9, 21.6), turned to 90 degrees
- moved SOURCE2 88.8 mm to (83.8, 20.3), turned to 90 degrees
- moved R12 87.6 mm to (22.9, 3.81)
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Connections:
- net N$13 renamed EXT_SOURCE
- removed net N$6: ON.K, R8.2
- new net N$11: R13.2, R15.1
- net GND: now also R14.1; no longer C1.-, R8.1
- net N$7: now also R14.2, R15.2; no longer R13.2
- net VCC: no longer C1.+, ON.A
Routing:
- net VCC: track 54.4 -> 181.8 mm, vias 0 -> 1
- net N$10: track 0.00 -> 89.1 mm
- net CURR_SENSE: track 0.00 -> 74.1 mm
- net GND: track 0.00 -> 73.2 mm, vias 0 -> 2
- net N$9: track 0.00 -> 70.2 mm, vias 0 -> 1
- net N$4: track 0.00 -> 48.1 mm
- net N$3: track 0.00 -> 47.9 mm
- net N$1: track 0.00 -> 36.9 mm
- net EXT_SOURCE: track 0.00 -> 34.9 mm
- net N$8: track 0.00 -> 32.4 mm
- net V-: track 10.2 -> 32.6 mm
- net N$7: track 0.00 -> 20.4 mm
- net N$5: track 0.00 -> 12.5 mm
- net N$2: track 0.00 -> 10.2 mm
- net N$11: track 0.00 -> 7.62 mm
- added copper zone on layer 16, net GND
Other:
- board size 160 x 100 mm -> 83.8 x 55.9 mm
- board text added: "+"
- board text added: "-"
- board text added: "- +"
- board text added: "Batt"
- board text added: "Coarse"
- board text added: "Ext"
- board text added: "Fine"
- board text added: "Nathan Campos, 2014"
- board text added: "Sense"
- board text added: "miniSource"
