File: Rev A.sch (EAGLE design)
At the start: 12 parts, among them IC1 LM324N, Q2 TIP41C

Commit message: Finished the schematic
Parts:
- removed IC1: LM324N, linear:LM324N
- added BAT1, BAT2: (no value), SparkFun-Electromechanical:BATTERYAA
- added C1: 47uF, rcl:CPOL-EUE2.5-6
- added C2, C3, C8: 0.1uF, rcl:C-EU050-025X075
- added C6: 10nF, rcl:C-EU050-025X075
- added C7: 100pF, rcl:C-EU025-025X050
- added C9: 100uF, rcl:CPOL-EUE2.5-6
- added D10, D9: 1N5817-B, diode:1N5817-B
- added IC2: NE555, st-microelectronics:NE555
- added IC3: LM358N, linear:LM358N
- added ON: (no value), led:LEDSQR2X5
- added R10, R9: 18kΩ, resistor:R-EU_0207/10
- added R11, R8: 1kΩ, resistor:R-EU_0207/10
- added R12: 5kΩ, bourns:3362U
- added R13: 100kΩ, bourns:3362U
- added R6: 4.7kΩ, resistor:R-EU_0207/10
- added R7: 10kΩ, resistor:R-EU_0207/10
- added RNG_SEL, SOURCE_SEL: (no value), pinhead:PINHD-2X2
- added SOURCE: M02JST-PTH-2, SparkFun-Connectors:M02JST-PTH-2
- added SOURCE1: (no value), pinhead:PINHD-1X2
- added SOURCE2: POWER_JACKPTH, SparkFun-Connectors:POWER_JACKPTH
Connections:
- new net N$10: BAT1.-, BAT2.+
- new net N$13: SOURCE.2, SOURCE1.2, SOURCE2.PWR, SOURCE_SEL.3
- new net N$17: C8.1, IC2.OUT
- new net N$18: C6.1, IC2.CON
- new net N$19: C7.1, IC2.TRE, IC2.TRI, R7.1
- new net N$20: IC2.DIS, R6.1, R7.2
- new net N$25: C8.2, D10.C, D9.A
- new net N$6: ON.C, R8.2
- new net N$8: IC3B.-IN, R10.1, R11.2, R9.1, RNG_SEL.1
- new net N$9: CURR_SENSE.1, IC3B.OUT, R10.2, R9.2, RNG_SEL.2
- new net V-: C9.-, D10.A, IC3P.V-
- new net VCC: BAT1.+, C1.+, C2.1, C3.1, IC2./RES, IC2.VCC+, IC3P.V+, ON.A, R13.3, R6.2, SOURCE_SEL.1
- net CURR_SENSE: now also IC3A.-IN, IC3B.+IN; no longer IC1A.-IN, IC1B.+IN
- net GND: now also BAT2.-, C1.-, C2.2, C3.2, C6.2, C7.2, C9.+, D9.C, IC2.GND, R11.1, R12.1, R8.1, SOURCE.1, SOURCE1.1, SOURCE2.GND, SOURCE2.GNDBREAK; no longer IC1P.V-
- net N$1: now also IC3A.OUT; no longer IC1A.OUT
- net N$3: now also SOURCE_SEL.2, SOURCE_SEL.4
- net N$5: now also R12.2, R13.1; no longer IC1B.-IN, IC1B.OUT
- net N$7: now also IC3A.+IN, R13.2; no longer IC1A.+IN
Other:
- note added: "1%"
- note added: "555 Timer"
- note added: "A"
- note added: "Coarse"
- note added: "Fine"
- note added: "Op-Amp"
- note added: "mA"
- note removed: "Use charge-pumps to generate the + and - supply rails for the op-amp?"
- note removed: "Use some sort of digital switch to switch between the internal and external power source for the current sourse part of the circuit using a single push button."
- moved on the sheet: CURR_SENSE, KK1

Commit message: Started laying out the board
Other:
- note added: "7555"
Changed lines of the file:
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@@
 <text x="10.16" y="40.64" size="1.778" layer="91" rot="R90" align="center">Fine</text>
 <text x="22.86" y="53.34" size="1.778" layer="91" rot="R90" align="center">Coarse</text>
+<text x="-15.24" y="-27.94" size="1.778" layer="91" align="center">7555</text>
 </plain>
 <instances>

Commit message: Made some little fixes to the schematic
Parts:
- added R14, R15: 100kΩ, resistor:R-EU_0207/10
Connections:
- net N$13 renamed EXT_SOURCE
- new net N$11: R13.2, R15.1
- net GND: now also R14.1
- net N$7: now also R14.2, R15.2; no longer R13.2
Other:
- moved on the sheet: R12, R13, SOURCE, SOURCE1, SOURCE2
Changed lines of the file:
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@@
 <part name="SUPPLY1" library="supply2" deviceset="V-" device=""/>
 <part name="P+5" library="supply1" deviceset="VCC" device=""/>
+<part name="R14" library="resistor" deviceset="R-EU_" device="0207/10" value="100kΩ"/>
+<part name="R15" library="resistor" deviceset="R-EU_" device="0207/10" value="100kΩ"/>
+<part name="GND14" library="supply1" deviceset="GND" device=""/>
 </parts>
 <sheets>
@@
 <text x="99.06" y="-15.24" size="1.778" layer="91" rot="R90" align="center">1%</text>
 <text x="-43.18" y="40.64" size="1.778" layer="91" rot="R90" align="center">Op-Amp</text>
-<text x="10.16" y="40.64" size="1.778" layer="91" rot="R90" align="center">Fine</text>
-<text x="22.86" y="53.34" size="1.778" layer="91" rot="R90" align="center">Coarse</text>
+<text x="-17.78" y="40.64" size="1.778" layer="91" rot="R90" align="center">Fine</text>
+<text x="-5.08" y="53.34" size="1.778" layer="91" rot="R90" align="center">Coarse</text>
 <text x="-15.24" y="-27.94" size="1.778" layer="91" align="center">7555</text>
 </plain>
@@
 <instance part="GND7" gate="1" x="-38.1" y="20.32"/>
 <instance part="P+6" gate="VCC" x="-38.1" y="58.42"/>
-<instance part="R12" gate="G$1" x="7.62" y="45.72"/>
-<instance part="R13" gate="G$1" x="20.32" y="58.42"/>
-<instance part="GND8" gate="1" x="7.62" y="30.48"/>
-<instance part="P+7" gate="VCC" x="20.32" y="73.66"/>
+<instance part="R12" gate="G$1" x="-20.32" y="45.72"/>
+<instance part="R13" gate="G$1" x="-7.62" y="58.42"/>
+<instance part="GND8" gate="1" x="-20.32" y="30.48"/>
+<instance part="P+7" gate="VCC" x="-7.62" y="73.66"/>
 <instance part="BAT1" gate="G$1" x="-99.06" y="45.72" rot="R270"/>
 <instance part="BAT2" gate="G$1" x="-99.06" y="33.02" rot="R270"/>
@@
 <instance part="SOURCE_SEL" gate="A" x="43.18" y="83.82"/>
 <instance part="P+9" gate="VCC" x="30.48" y="101.6"/>
-<instance part="SOURCE" gate="G$1" x="-25.4" y="81.28"/>
-<instance part="SOURCE1" gate="G$1" x="-5.08" y="93.98" rot="R90"/>
-<instance part="GND25" gate="1" x="5.08" y="71.12"/>
-<instance part="SOURCE2" gate="G$1" x="-17.78" y="60.96"/>
-<instance part="GND13" gate="1" x="-12.7" y="53.34"/>
+<instance part="SOURCE" gate="G$1" x="-88.9" y="-10.16"/>
+<instance part="SOURCE1" gate="G$1" x="-68.58" y="2.54" rot="R90"/>
+<instance part="GND25" gate="1" x="-58.42" y="-20.32"/>
+<instance part="SOURCE2" gate="G$1" x="-81.28" y="-30.48"/>
+<instance part="GND13" gate="1" x="-76.2" y="-38.1"/>
 <instance part="IC3" gate="A" x="38.1" y="55.88"/>
 <instance part="IC3" gate="B" x="111.76" y="12.7"/>
@@
 <instance part="SUPPLY1" gate="1" x="38.1" y="45.72"/>
 <instance part="P+5" gate="VCC" x="38.1" y="66.04"/>
+<instance part="R14" gate="G$1" x="22.86" y="45.72" rot="R90"/>
+<instance part="R15" gate="G$1" x="10.16" y="58.42"/>
+<instance part="GND14" gate="1" x="22.86" y="30.48"/>
 </instances>
 <busses>
@@
 <pinref part="GND8" gate="1" pin="GND"/>
 <pinref part="R12" gate="G$1" pin="1"/>
-<wire x1="7.62" y1="33.02" x2="7.62" y2="40.64" width="0.1524" layer="91"/>
+<wire x1="-20.32" y1="33.02" x2="-20.32" y2="40.64" width="0.1524" layer="91"/>
 </segment>
 <segment>
@@
 </segment>
 <segment>
-<wire x1="5.08" y1="81.28" x2="5.08" y2="73.66" width="0.1524" layer="91"/>
+<wire x1="-58.42" y1="-10.16" x2="-58.42" y2="-17.78" width="0.1524" layer="91"/>
 <pinref part="SOURCE" gate="G$1" pin="1"/>
-<wire x1="5.08" y1="81.28" x2="-7.62" y2="81.28" width="0.1524" layer="91"/>
+<wire x1="-58.42" y1="-10.16" x2="-71.12" y2="-10.16" width="0.1524" layer="91"/>
 <pinref part="SOURCE1" gate="G$1" pin="1"/>
-<wire x1="-7.62" y1="81.28" x2="-17.78" y2="81.28" width="0.1524" layer="91"/>
-<wire x1="-7.62" y1="91.44" x2="-7.62" y2="81.28" width="0.1524" layer="91"/>
-<junction x="-7.62" y="81.28"/>
+<wire x1="-71.12" y1="-10.16" x2="-81.28" y2="-10.16" width="0.1524" layer="91"/>
+<wire x1="-71.12" y1="0" x2="-71.12" y2="-10.16" width="0.1524" layer="91"/>
+<junction x="-71.12" y="-10.16"/>
 <pinref part="GND25" gate="1" pin="GND"/>
 </segment>
 <segment>
 <pinref part="SOURCE2" gate="G$1" pin="GND"/>
-<wire x1="-15.24" y1="63.5" x2="-12.7" y2="63.5" width="0.1524" layer="91"/>
-<wire x1="-12.7" y1="63.5" x2="-12.7" y2="66.04" width="0.1524" layer="91"/>
+<wire x1="-78.74" y1="-27.94" x2="-76.2" y2="-27.94" width="0.1524" layer="91"/>
+<wire x1="-76.2" y1="-27.94" x2="-76.2" y2="-25.4" width="0.1524" layer="91"/>
 <pinref part="SOURCE2" gate="G$1" pin="GNDBREAK"/>
-<wire x1="-12.7" y1="66.04" x2="-15.24" y2="66.04" width="0.1524" layer="91"/>
-<wire x1="-12.7" y1="63.5" x2="-12.7" y2="55.88" width="0.1524" layer="91"/>
-<junction x="-12.7" y="63.5"/>
+<wire x1="-76.2" y1="-25.4" x2="-78.74" y2="-25.4" width="0.1524" layer="91"/>
+<wire x1="-76.2" y1="-27.94" x2="-76.2" y2="-35.56" width="0.1524" layer="91"/>
+<junction x="-76.2" y="-27.94"/>
 <pinref part="GND13" gate="1" pin="GND"/>
+</segment>
+<segment>
+<pinref part="R14" gate="G$1" pin="1"/>
+<wire x1="22.86" y1="40.64" x2="22.86" y2="33.02" width="0.1524" layer="91"/>
+<pinref part="GND14" gate="1" pin="GND"/>
 </segment>
 </net>
@@
 </segment>
 </net>
-<net name="N$7" class="0">
-<segment>
-<wire x1="30.48" y1="58.42" x2="25.4" y2="58.42" width="0.1524" layer="91"/>
-<pinref part="R13" gate="G$1" pin="2"/>
-<pinref part="IC3" gate="A" pin="+IN"/>
-</segment>
-</net>
 <net name="N$17" class="0">
 <segment>
@@
 <pinref part="R13" gate="G$1" pin="3"/>
 <pinref part="P+7" gate="VCC" pin="VCC"/>
-<wire x1="20.32" y1="63.5" x2="20.32" y2="71.12" width="0.1524" layer="91"/>
+<wire x1="-7.62" y1="63.5" x2="-7.62" y2="71.12" width="0.1524" layer="91"/>
 </segment>
 <segment>
@@
 <pinref part="R12" gate="G$1" pin="2"/>
 <pinref part="R13" gate="G$1" pin="1"/>
-<wire x1="12.7" y1="45.72" x2="20.32" y2="45.72" width="0.1524" layer="91"/>
-<wire x1="20.32" y1="45.72" x2="20.32" y2="53.34" width="0.1524" layer="91"/>
+<wire x1="-15.24" y1="45.72" x2="-7.62" y2="45.72" width="0.1524" layer="91"/>
+<wire x1="-7.62" y1="45.72" x2="-7.62" y2="53.34" width="0.1524" layer="91"/>
 </segment>
 </net>
@@
 </segment>
 </net>
-<net name="N$13" class="0">
+<net name="N$7" class="0">
+<segment>
+<pinref part="R15" gate="G$1" pin="2"/>
+<pinref part="IC3" gate="A" pin="+IN"/>
+<wire x1="15.24" y1="58.42" x2="22.86" y2="58.42" width="0.1524" layer="91"/>
+<pinref part="R14" gate="G$1" pin="2"/>
+<wire x1="22.86" y1="58.42" x2="30.48" y2="58.42" width="0.1524" layer="91"/>
+<wire x1="22.86" y1="50.8" x2="22.86" y2="58.42" width="0.1524" layer="91"/>
+<junction x="22.86" y="58.42"/>
+</segment>
+</net>
+<net name="N$11" class="0">
+<segment>
+<pinref part="R13" gate="G$1" pin="2"/>
+<pinref part="R15" gate="G$1" pin="1"/>
+<wire x1="-2.54" y1="58.42" x2="5.08" y2="58.42" width="0.1524" layer="91"/>
+</segment>
+</net>
+<net name="EXT_SOURCE" class="0">
 <segment>
 <pinref part="SOURCE_SEL" gate="A" pin="3"/>
+<wire x1="38.1" y1="83.82" x2="22.86" y2="83.82" width="0.1524" layer="91"/>
+<label x="25.4" y="86.36" size="1.778" layer="95" rot="R180"/>
+</segment>
+<segment>
 <pinref part="SOURCE" gate="G$1" pin="2"/>
-<wire x1="38.1" y1="83.82" x2="-5.08" y2="83.82" width="0.1524" layer="91"/>
 <pinref part="SOURCE1" gate="G$1" pin="2"/>
-<wire x1="-5.08" y1="83.82" x2="-17.78" y2="83.82" width="0.1524" layer="91"/>
-<wire x1="-5.08" y1="91.44" x2="-5.08" y2="83.82" width="0.1524" layer="91"/>
-<junction x="-5.08" y="83.82"/>
+<wire x1="-68.58" y1="-7.62" x2="-81.28" y2="-7.62" width="0.1524" layer="91"/>
+<wire x1="-68.58" y1="0" x2="-68.58" y2="-7.62" width="0.1524" layer="91"/>
+<junction x="-68.58" y="-7.62"/>
 <pinref part="SOURCE2" gate="G$1" pin="PWR"/>
-<wire x1="-15.24" y1="68.58" x2="-5.08" y2="68.58" width="0.1524" layer="91"/>
-<wire x1="-5.08" y1="68.58" x2="-5.08" y2="83.82" width="0.1524" layer="91"/>
-</segment>
-</net>
+<wire x1="-78.74" y1="-22.86" x2="-68.58" y2="-22.86" width="0.1524" layer="91"/>
+<wire x1="-68.58" y1="-22.86" x2="-68.58" y2="-7.62" width="0.1524" layer="91"/>
+<wire x1="-68.58" y1="-7.62" x2="-58.42" y2="-7.62" width="0.1524" layer="91"/>
+<label x="-45.72" y="-5.08" size="1.778" layer="95" rot="R180"/>
+</segment>
+</net>

Commit message: Finished the layout
Parts:
- removed C1: 47uF, rcl:CPOL-EUE2.5-6
- removed ON: (no value), led:LEDSQR2X5
- removed R8: 1kΩ, resistor:R-EU_0207/10
Connections:
- removed net N$6: ON.C, R8.2
- net GND: no longer C1.-, R8.1
- net VCC: no longer C1.+, ON.A
Other:
- moved on the sheet: BAT1, BAT2, C2, C3
Changed lines of the file:
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@@
 <part name="P+1" library="supply1" deviceset="VCC" device=""/>
 <part name="P+2" library="supply1" deviceset="VCC" device=""/>
-<part name="GND4" library="supply1" deviceset="GND" device=""/>
-<part name="P+3" library="supply1" deviceset="VCC" device=""/>
-<part name="ON" library="led" deviceset="LED" device="SQR2X5"/>
-<part name="R8" library="resistor" deviceset="R-EU_" device="0207/10" value="1kΩ"/>
-<part name="C1" library="rcl" deviceset="CPOL-EU" device="E2.5-6" value="47uF"/>
-<part name="P+4" library="supply1" deviceset="VCC" device=""/>
-<part name="GND6" library="supply1" deviceset="GND" device=""/>
 <part name="C8" library="rcl" deviceset="C-EU" device="050-025X075" value="0.1uF"/>
 <part name="SUPPLY2" library="supply2" deviceset="V-" device=""/>
@@
 <sheet>
 <plain>
-<text x="-58.42" y="40.64" size="1.778" layer="91" rot="R90" align="center">555 Timer</text>
+<text x="-66.04" y="40.64" size="1.778" layer="91" rot="R90" align="center">555 Timer</text>
 <text x="129.54" y="-20.32" size="1.778" layer="91" align="center">mA</text>
 <text x="129.54" y="-17.78" size="1.778" layer="91" align="center">A</text>
 <text x="99.06" y="-15.24" size="1.778" layer="91" rot="R90" align="center">1%</text>
-<text x="-43.18" y="40.64" size="1.778" layer="91" rot="R90" align="center">Op-Amp</text>
+<text x="-50.8" y="40.64" size="1.778" layer="91" rot="R90" align="center">Op-Amp</text>
 <text x="-17.78" y="40.64" size="1.778" layer="91" rot="R90" align="center">Fine</text>
 <text x="-5.08" y="53.34" size="1.778" layer="91" rot="R90" align="center">Coarse</text>
@@
 <instance part="CURR_SENSE" gate="G$1" x="142.24" y="10.16"/>
 <instance part="GND1" gate="1" x="132.08" y="-2.54"/>
-<instance part="C3" gate="G$1" x="-53.34" y="40.64"/>
-<instance part="GND5" gate="1" x="-53.34" y="20.32"/>
+<instance part="C3" gate="G$1" x="-60.96" y="40.64"/>
+<instance part="GND5" gate="1" x="-60.96" y="20.32"/>
 <instance part="IC2" gate="G$1" x="-15.24" y="-12.7"/>
 <instance part="C6" gate="G$1" x="2.54" y="-25.4"/>
@@
 <instance part="GND18" gate="1" x="17.78" y="-43.18"/>
 <instance part="P+1" gate="VCC" x="-20.32" y="20.32"/>
-<instance part="P+2" gate="VCC" x="-53.34" y="58.42"/>
-<instance part="GND4" gate="1" x="-83.82" y="20.32"/>
-<instance part="P+3" gate="VCC" x="-83.82" y="58.42"/>
-<instance part="ON" gate="G$1" x="-83.82" y="48.26"/>
-<instance part="R8" gate="G$1" x="-83.82" y="33.02" rot="R90"/>
-<instance part="C1" gate="G$1" x="-68.58" y="40.64"/>
-<instance part="P+4" gate="VCC" x="-68.58" y="58.42"/>
-<instance part="GND6" gate="1" x="-68.58" y="20.32"/>
+<instance part="P+2" gate="VCC" x="-60.96" y="58.42"/>
 <instance part="C8" gate="G$1" x="5.08" y="-12.7" rot="R90"/>
 <instance part="SUPPLY2" gate="1" x="38.1" y="2.54" rot="R180"/>
@@
 <instance part="R11" gate="G$1" x="96.52" y="-17.78" rot="R90"/>
 <instance part="GND2" gate="1" x="96.52" y="-35.56"/>
-<instance part="C2" gate="G$1" x="-38.1" y="40.64"/>
-<instance part="GND7" gate="1" x="-38.1" y="20.32"/>
-<instance part="P+6" gate="VCC" x="-38.1" y="58.42"/>
+<instance part="C2" gate="G$1" x="-45.72" y="40.64"/>
+<instance part="GND7" gate="1" x="-45.72" y="20.32"/>
+<instance part="P+6" gate="VCC" x="-45.72" y="58.42"/>
 <instance part="R12" gate="G$1" x="-20.32" y="45.72"/>
 <instance part="R13" gate="G$1" x="-7.62" y="58.42"/>
 <instance part="GND8" gate="1" x="-20.32" y="30.48"/>
 <instance part="P+7" gate="VCC" x="-7.62" y="73.66"/>
-<instance part="BAT1" gate="G$1" x="-99.06" y="45.72" rot="R270"/>
-<instance part="BAT2" gate="G$1" x="-99.06" y="33.02" rot="R270"/>
-<instance part="P+8" gate="VCC" x="-99.06" y="58.42"/>
-<instance part="GND12" gate="1" x="-99.06" y="20.32"/>
+<instance part="BAT1" gate="G$1" x="-76.2" y="45.72" rot="R270"/>
+<instance part="BAT2" gate="G$1" x="-76.2" y="33.02" rot="R270"/>
+<instance part="P+8" gate="VCC" x="-76.2" y="58.42"/>
+<instance part="GND12" gate="1" x="-76.2" y="20.32"/>
 <instance part="SOURCE_SEL" gate="A" x="43.18" y="83.82"/>
 <instance part="P+9" gate="VCC" x="30.48" y="101.6"/>
@@
 <segment>
 <pinref part="C3" gate="G$1" pin="2"/>
-<wire x1="-53.34" y1="35.56" x2="-53.34" y2="22.86" width="0.1524" layer="91"/>
+<wire x1="-60.96" y1="35.56" x2="-60.96" y2="22.86" width="0.1524" layer="91"/>
 <pinref part="GND5" gate="1" pin="GND"/>
 </segment>
@@
 </segment>
 <segment>
-<wire x1="-83.82" y1="22.86" x2="-83.82" y2="27.94" width="0.1524" layer="91"/>
-<pinref part="GND4" gate="1" pin="GND"/>
-<pinref part="R8" gate="G$1" pin="1"/>
-</segment>
-<segment>
-<pinref part="C1" gate="G$1" pin="-"/>
-<wire x1="-68.58" y1="35.56" x2="-68.58" y2="22.86" width="0.1524" layer="91"/>
-<pinref part="GND6" gate="1" pin="GND"/>
-</segment>
-<segment>
 <pinref part="R11" gate="G$1" pin="1"/>
 <wire x1="96.52" y1="-22.86" x2="96.52" y2="-33.02" width="0.1524" layer="91"/>
@@
 <segment>
 <pinref part="C2" gate="G$1" pin="2"/>
-<wire x1="-38.1" y1="35.56" x2="-38.1" y2="22.86" width="0.1524" layer="91"/>
+<wire x1="-45.72" y1="35.56" x2="-45.72" y2="22.86" width="0.1524" layer="91"/>
 <pinref part="GND7" gate="1" pin="GND"/>
 </segment>
@@
 <pinref part="BAT2" gate="G$1" pin="-"/>
 <pinref part="GND12" gate="1" pin="GND"/>
-<wire x1="-99.06" y1="27.94" x2="-99.06" y2="22.86" width="0.1524" layer="91"/>
+<wire x1="-76.2" y1="27.94" x2="-76.2" y2="22.86" width="0.1524" layer="91"/>
 </segment>
 <segment>
@@
 <segment>
 <pinref part="C3" gate="G$1" pin="1"/>
-<wire x1="-53.34" y1="43.18" x2="-53.34" y2="55.88" width="0.1524" layer="91"/>
+<wire x1="-60.96" y1="43.18" x2="-60.96" y2="55.88" width="0.1524" layer="91"/>
 <pinref part="P+2" gate="VCC" pin="VCC"/>
 </segment>
 <segment>
-<wire x1="-83.82" y1="50.8" x2="-83.82" y2="55.88" width="0.1524" layer="91"/>
-<pinref part="P+3" gate="VCC" pin="VCC"/>
-<pinref part="ON" gate="G$1" pin="A"/>
-</segment>
-<segment>
-<pinref part="C1" gate="G$1" pin="+"/>
-<wire x1="-68.58" y1="43.18" x2="-68.58" y2="55.88" width="0.1524" layer="91"/>
-<pinref part="P+4" gate="VCC" pin="VCC"/>
-</segment>
-<segment>
 <pinref part="C2" gate="G$1" pin="1"/>
-<wire x1="-38.1" y1="43.18" x2="-38.1" y2="55.88" width="0.1524" layer="91"/>
+<wire x1="-45.72" y1="43.18" x2="-45.72" y2="55.88" width="0.1524" layer="91"/>
 <pinref part="P+6" gate="VCC" pin="VCC"/>
 </segment>
@@
 <segment>
 <pinref part="BAT1" gate="G$1" pin="+"/>
-<wire x1="-99.06" y1="50.8" x2="-99.06" y2="55.88" width="0.1524" layer="91"/>
+<wire x1="-76.2" y1="50.8" x2="-76.2" y2="55.88" width="0.1524" layer="91"/>
 <pinref part="P+8" gate="VCC" pin="VCC"/>
 </segment>
@@
 <pinref part="IC3" gate="P" pin="V+"/>
 <pinref part="P+5" gate="VCC" pin="VCC"/>
-</segment>
-</net>
-<net name="N$6" class="0">
-<segment>
-<wire x1="-83.82" y1="43.18" x2="-83.82" y2="38.1" width="0.1524" layer="91"/>
-<pinref part="R8" gate="G$1" pin="2"/>
-<pinref part="ON" gate="G$1" pin="C"/>
 </segment>
 </net>
@@
 <pinref part="BAT1" gate="G$1" pin="-"/>
 <pinref part="BAT2" gate="G$1" pin="+"/>
-<wire x1="-99.06" y1="40.64" x2="-99.06" y2="38.1" width="0.1524" layer="91"/>
-</segment>
-</net>
+<wire x1="-76.2" y1="40.64" x2="-76.2" y2="38.1" width="0.1524" layer="91"/>
+</segment>
+</net>
